File: variable load.kicad_pcb (KiCad board)
At the start: 2 copper layers, 130.2 x 99.2 mm, 42 parts, among them IC1 OPA4197ID, IC2 OPA4197ID, J1 Screw_Terminal_01x02, J2 Screw_Terminal_01x03, J3 Screw_Terminal_01x02, Q1 IXTX110N20L2, Q2 IXTX110N20L2, Q3 IXTX110N20L2, Q4 IXTX110N20L2, Q5 IXTX110N20L2, Q6 IXTX110N20L2, Q7 IXTX110N20L2, Q8 IXTX110N20L2

Commit message: layout question
Parts:
- added C13: 470p, Capacitor_SMD:C_0805_2012Metric, F.Cu at (96.3, 78.0)
- added C14: 470p, Capacitor_SMD:C_0805_2012Metric, F.Cu at (158.7, 114.9)
- added C15: 100nF, Capacitor_SMD:C_0805_2012Metric, F.Cu at (82.3, 99.4)
- added C16: 100nF, Capacitor_SMD:C_0805_2012Metric, F.Cu at (82.3, 102.4)
- added C17: 100nF, Capacitor_SMD:C_0805_2012Metric, F.Cu at (82.3, 105.4)
- added C18: 470p, Capacitor_SMD:C_0805_2012Metric, F.Cu at (82.3, 108.4)
- added C19: 1uF, Capacitor_SMD:C_0805_2012Metric, F.Cu at (82.3, 111.4)
- added C20: 470p, Capacitor_SMD:C_0805_2012Metric, F.Cu at (82.3, 114.5)
- added C21: 10uF, Capacitor_SMD:C_0805_2012Metric, F.Cu at (82.3, 117.5)
- added IC3: OPA4197ID, Package_SO:SOIC-14_3.9x8.7mm_P1.27mm, F.Cu at (125.2, 112.1)
- added Q10: IXTX110N20L2, Package_TO_SOT_THT:TO-247-3_Vertical, B.Cu at (80.0, 143.5)
- added Q9: IXTX110N20L2, Package_TO_SOT_THT:TO-247-3_Vertical, B.Cu at (59.0, 143.9)
- added R18: 100, Resistor_SMD:R_0805_2012Metric, F.Cu at (152.2, 104.4)
- added R19: 0.05, Resistor_SMD:R_2512_6332Metric, F.Cu at (70.0, 131.5)
- added R20: 0.05, Resistor_SMD:R_2512_6332Metric, F.Cu at (144.3, 84.1)
- added R21: 100k, Resistor_SMD:R_0805_2012Metric, F.Cu at (109.6, 71.9)
- added R22: 100k, Resistor_SMD:R_0805_2012Metric, F.Cu at (109.6, 74.8)
- added R23: 0.05, Resistor_SMD:R_2512_6332Metric, F.Cu at (100.0, 130.7)
- added R24: 0.05, Resistor_SMD:R_2512_6332Metric, F.Cu at (144.3, 89.0)
- added R25: 1k, Resistor_SMD:R_0805_2012Metric, F.Cu at (181.0, 76.9)
- added R26: 1k, Resistor_SMD:R_0805_2012Metric, F.Cu at (198.0, 77.4)
- added R27: 1k, Resistor_SMD:R_0805_2012Metric, F.Cu at (217.8, 62.6)
- added R28: 0.05, Resistor_SMD:R_2512_6332Metric, F.Cu at (124.5, 134.0)
- added R29: 100k, Resistor_SMD:R_0805_2012Metric, F.Cu at (165.4, 107.5)
- added R30: 0.05, Resistor_SMD:R_2512_6332Metric, F.Cu at (145.0, 136.0)
- added R31: 100, Resistor_SMD:R_0805_2012Metric, F.Cu at (164.8, 116.9)
- added R32: 100k, Resistor_SMD:R_0805_2012Metric, F.Cu at (70.1, 119.2)
- added R33: 100, Resistor_SMD:R_0805_2012Metric, F.Cu at (70.1, 122.1)
- added R34: 10k, Resistor_SMD:R_0805_2012Metric, F.Cu at (194.0, 90.9)
- added R35: 3.48M, Resistor_SMD:R_1206_3216Metric, F.Cu at (187.5, 100.4)
- added R36: 1k, Resistor_SMD:R_0805_2012Metric, F.Cu at (195.8, 98.9)
- added R37: 6.98k, Resistor_SMD:R_0805_2012Metric, F.Cu at (195.8, 101.9)
- added U1: R-78HE5.0-0.3, footprints:SIP900W75P254L1200H1300Q3, F.Cu at (68.8, 87.5)
- added U2: 6N137, Package_DIP:DIP-8_W7.62mm, F.Cu at (170.0, 73.1)
- added U3: 6N137, Package_DIP:DIP-8_W7.62mm, F.Cu at (186.7, 73.4)
- added U4: 6N137, Package_DIP:DIP-8_W7.62mm, F.Cu at (203.2, 73.6)
- added U5: MCP4822-E_MS, footprints:SOP65P490X110-8N, F.Cu at (186.0, 90.9)
- C1: value 1u -> 10uF
- C11, C9: value 1u -> 470p
- C2: value 1u -> 100nF
- C3, C4: value 470p -> 10uF
- C7, C8: value 470p -> 1uF
- J1: footprint TerminalBlock_Phoenix:TerminalBlock_Phoenix_MKDS-1,5-2_1x02_P5.00mm_Horizontal -> TerminalBlock_Phoenix:TerminalBlock_Phoenix_MKDS-3-2-5.08_1x02_P5.08mm_Horizontal
- J2: value Screw_Terminal_01x03 -> Screw_Terminal_01x02; footprint TerminalBlock_Phoenix:TerminalBlock_Phoenix_MKDS-1,5-3_1x03_P5.00mm_Horizontal -> TerminalBlock_Phoenix:TerminalBlock_Phoenix_MKDS-3-2-5.08_1x02_P5.08mm_Horizontal
- J3: value Screw_Terminal_01x02 -> Conn_01x04; footprint TerminalBlock_Phoenix:TerminalBlock_Phoenix_MKDS-1,5-2_1x02_P5.00mm_Horizontal -> Connector_JST:JST_XH_B4B-XH-A_1x04_P2.50mm_Vertical
- R10, R16, R3, R9: value 0.05 -> 100k; footprint Resistor_SMD:R_2512_6332Metric -> Resistor_SMD:R_0805_2012Metric
- R14, R7: value 0.05 -> 100; footprint Resistor_SMD:R_2512_6332Metric -> Resistor_SMD:R_0805_2012Metric
- R15, R4: value 100 -> 100k
- R17: value 1 -> 100; footprint Resistor_SMD:R_2512_6332Metric -> Resistor_SMD:R_0805_2012Metric
- R2, R6: value 100 -> 0.05; footprint Resistor_SMD:R_0805_2012Metric -> Resistor_SMD:R_2512_6332Metric
- moved R5 193.0 mm to (218.0, 130.5)
- moved Q4 161.9 mm to (161.1, 144.5), turned to 0 degrees
- moved R1 155.7 mm to (191.5, 132.5)
- moved J3 134.1 mm to (186.6, 62.7), turned to 0 degrees
- moved Q3 132.1 mm to (139.1, 144.0), turned to 0 degrees
- moved R2 129.3 mm to (165.5, 132.9), turned to 0 degrees
- moved Q5 110.6 mm to (186.1, 142.5), turned to 0 degrees
- moved Q2 101.5 mm to (116.5, 142.8), turned to 0 degrees
- moved R6 94.9 mm to (112.5, 126.7), turned to 0 degrees
- moved Q7 88.8 mm to (213.6, 142.3), turned to 0 degrees
- moved IC1 84.4 mm to (139.7, 112.9)
- moved J1 83.9 mm to (68.3, 60.5), turned to 90 degrees
- moved C8 78.1 mm to (158.7, 108.9)
- moved Q1 71.3 mm to (93.6, 143.4), turned to 0 degrees
- moved R7 70.6 mm to (100.7, 71.9)
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Connections:
- C1 pad 1: GND -> 12V
- C1 pad 2: +12V -> GND
- C10 pad 1: Net-(IC2--IN_D) -> Net-(IC2--IN_A)
- C10 pad 2: Net-(IC2-OUT_D) -> Net-(IC2-OUT_A)
- C11 pad 1: -12V -> Net-(IC1--IN_D)
- C11 pad 2: GND -> Net-(IC1-OUT_D)
- C12 pad 1: Net-(IC2--INC) -> Net-(IC2--IN_D)
- C12 pad 2: Net-(IC2-OUTC) -> Net-(IC2-OUT_D)
- C2 pad 1: -12V -> 5V_LOAD
- C3 pad 1: Net-(IC1--IN_A) -> 5V_LOAD
- C3 pad 2: Net-(IC1-OUT_A) -> GND
- C4 pad 1: Net-(IC1--INB) -> 5V_LOAD
- C4 pad 2: Net-(IC1-OUTB) -> GND
- C5 pad 1: Net-(IC1--INC) -> Net-(IC1--INB)
- C5 pad 2: Net-(IC1-OUTC) -> Net-(IC1-OUTB)
- C6 pad 1: Net-(IC1--IN_D) -> Net-(IC2--INB)
- C6 pad 2: Net-(IC1-OUT_D) -> Net-(IC2-OUTB)
- C7 pad 1: Net-(IC2--INB) -> GND
- C7 pad 2: Net-(IC2-OUTB) -> 12V
- C8 pad 1: Net-(IC2--IN_A) -> GND
- C8 pad 2: Net-(IC2-OUT_A) -> 12V
- C9 pad 1: GND -> Net-(IC1--IN_A)
- C9 pad 2: +12V -> Net-(IC1-OUT_A)
- IC1 pad 10: /Vref -> VREF
- IC1 pad 11: -12V -> GND
- IC1 pad 12: /Vref -> VREF
- IC1 pad 3: /Vref -> VREF
- IC1 pad 4: +12V -> 12V
- IC1 pad 5: /Vref -> VREF
- IC2 pad 10: /Vref -> VREF
- IC2 pad 11: -12V -> GND
- IC2 pad 12: /Vref -> VREF
- IC2 pad 3: /Vref -> VREF
- IC2 pad 4: +12V -> 12V
- IC2 pad 5: /Vref -> VREF
- J1 pad 1: Net-(J1-Pin_1) -> GND
- J1 pad 2: GND -> VTURB
- J2 pad 1: +12V -> GND
- J2 pad 2: GND -> 12V
- J3 pad 1: /Vref -> 5V_LED
- J3 pad 2: GND -> SCK_K
- Q1 pad 2: /Vturb -> VTURB
- Q1 pad 3: Net-(IC1--IN_A) -> Net-(IC1--INB)
- Q2 pad 2: /Vturb -> VTURB
- Q2 pad 3: Net-(IC1--INB) -> Net-(IC2--INB)
- Q3 pad 2: /Vturb -> VTURB
- Q3 pad 3: Net-(IC1--INC) -> Net-(IC1--IN_A)
- Q4 pad 2: /Vturb -> VTURB
- Q4 pad 3: Net-(IC1--IN_D) -> Net-(IC2--IN_A)
- Q5 pad 2: /Vturb -> VTURB
- Q5 pad 3: Net-(IC2--INB) -> Net-(IC1--IN_D)
- Q6 pad 2: /Vturb -> VTURB
- Q6 pad 3: Net-(IC2--IN_A) -> Net-(IC2--IN_D)
- Q7 pad 2: /Vturb -> VTURB
- Q7 pad 3: Net-(IC2--IN_D) -> Net-(IC1--INC)
- Q8 pad 2: /Vturb -> VTURB
- R1 pad 1: Net-(IC1--IN_A) -> Net-(IC1--INB)
- R10 pad 1: Net-(IC2--IN_A) -> Net-(Q4-G)
- R11 pad 1: Net-(IC2-OUTB) -> Net-(IC1-OUT_A)
- R11 pad 2: Net-(Q5-G) -> Net-(Q3-G)
- R12 pad 2: Net-(Q6-G) -> Net-(Q4-G)
- R13 pad 1: Net-(IC2-OUT_D) -> Net-(IC1-OUT_D)
- R13 pad 2: Net-(Q7-G) -> Net-(Q5-G)
- R14 pad 1: Net-(IC2--IN_D) -> Net-(IC2-OUT_D)
- R14 pad 2: GND -> Net-(Q6-G)
- R15 pad 1: Net-(IC2-OUTC) -> Net-(Q5-G)
- R15 pad 2: Net-(Q8-G) -> GND
- R16 pad 1: Net-(IC2--INC) -> Net-(Q6-G)
- R17 pad 1: /Vturb -> Net-(IC1-OUTC)
- R17 pad 2: Net-(J1-Pin_1) -> Net-(Q7-G)
- R2 pad 1: Net-(IC1-OUT_A) -> Net-(IC2--INB)
- R2 pad 2: Net-(Q1-G) -> GND
- R3 pad 1: Net-(IC1--INB) -> GND
- R3 pad 2: GND -> Net-(Q1-G)
- R4 pad 1: Net-(IC1-OUTB) -> GND
- R5 pad 1: Net-(IC1--INC) -> Net-(IC1--IN_A)
- R6 pad 1: Net-(IC1-OUTC) -> Net-(IC2--IN_A)
- R6 pad 2: Net-(Q3-G) -> GND
- R7 pad 1: Net-(IC1--IN_D) -> Net-(IC1-OUTB)
- R7 pad 2: GND -> Net-(Q1-G)
- R8 pad 1: Net-(IC1-OUT_D) -> Net-(IC2-OUTB)
- R8 pad 2: Net-(Q4-G) -> Net-(Q2-G)
- R9 pad 1: Net-(IC2--INB) -> Net-(Q3-G)
Routing:
- net /Vturb: track 312.5 -> 0.00 mm, vias 2 -> 0
- net +12V: track 221.2 -> 0.00 mm, vias 4 -> 0
- net Net-(IC1-OUT_A): track 164.5 -> 0.00 mm
- net /Vref: track 124.9 -> 0.00 mm
- net Net-(IC1--IN_A): track 124.0 -> 0.00 mm
- net Net-(IC2--INB): track 121.6 -> 0.00 mm
- net -12V: track 114.9 -> 0.00 mm, vias 4 -> 0
- net Net-(IC2-OUTB): track 106.8 -> 0.00 mm
- net Net-(IC1--IN_D): track 95.4 -> 0.00 mm
- net Net-(IC2--IN_A): track 88.6 -> 0.00 mm, vias 2 -> 0
- net Net-(IC2--INC): track 71.7 -> 0.00 mm
- net GND: track 69.2 -> 0.00 mm, vias 28 -> 0
- net Net-(IC1--INC): track 60.1 -> 0.00 mm, vias 2 -> 0
- net Net-(IC2-OUT_A): track 56.9 -> 0.00 mm
- net Net-(IC2-OUTC): track 54.2 -> 0.00 mm
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- removed copper zone on B.Cu, net GND
Other:
- board outline removed
