File: variable load.kicad_sch (KiCad schematic)
At the start: 65 parts, among them IC1 OPA4197ID, IC2 OPA4197ID, IC3 OPA4197ID, J1 Screw_Terminal_01x02, J2 Screw_Terminal_01x03, J3 Screw_Terminal_01x02, J4 Conn_01x04, Q1 IXTX110N20L2, Q2 IXTX110N20L2, Q3 IXTX110N20L2, Q4 IXTX110N20L2, Q5 IXTX110N20L2, Q6 IXTX110N20L2, Q7 IXTX110N20L2, Q8 IXTX110N20L2, U1 MCP4822-E_MS, U2 6N137, U3 R-78HE5.0-0.3, U7 6N137, U8 6N137

Commit message: layout question
Parts:
- removed C1, C2, C20, C21: 1u, Capacitor_SMD:C_0805_2012Metric, symbol Device:C_US
- removed C13, C17, C18, C19: 100nF, symbol Device:C
- removed C14, C22: 10uF, symbol Device:C
- removed C15, C16: 10uF, Package_SO:SOIC-8_3.9x4.9mm_P1.27mm, symbol Device:C
- removed C3, C4, C8: 470p, Capacitor_SMD:C_0805_2012Metric, symbol Device:C_US
- removed IC3: OPA4197ID, Package_SO:SOIC-14_3.9x8.7mm_P1.27mm, symbol OPA4172IDR:OPA4172IDR
- removed J2: Screw_Terminal_01x03, TerminalBlock_Phoenix:TerminalBlock_Phoenix_MKDS-1,5-3_1x03_P5.00mm_Horizontal, symbol Connector:Screw_Terminal_01x03
- removed J3: Screw_Terminal_01x02, TerminalBlock_Phoenix:TerminalBlock_Phoenix_MKDS-1,5-2_1x02_P5.00mm_Horizontal, symbol Connector:Screw_Terminal_01x02
- removed J4: Conn_01x04, symbol Connector_Generic:Conn_01x04
- removed Q6: IXTX110N20L2, Package_TO_SOT_THT:TO-247-3_Vertical, symbol Transistor_FET:Q_NMOS_GDS
- removed R10, R3, R9: 0.05, Resistor_SMD:R_2512_6332Metric, symbol Device:R_US
- removed R24, R26, R29: 1k, symbol Device:R
- removed R27: 10k, symbol Device:R
- removed R28: 6.98k, symbol Device:R
- removed R4: 100, Resistor_SMD:R_0805_2012Metric, symbol Device:R_US
- removed U1: MCP4822-E_MS, MCP4822-E_MS:SOP65P490X110-8N, symbol MCP4822-E_MS:MCP4822-E_MS
- removed U2, U7, U8: 6N137, Package_DIP:DIP-8_W7.62mm, symbol Isolator:6N137
- removed U3: R-78HE5.0-0.3, R-78HE5.0-0.3:SIP900W75P254L1200H1300Q3, symbol R-78HE5.0-0.3:R-78HE5.0-0.3
- added C1, C3, C4: 10uF, Capacitor_SMD:C_0805_2012Metric, symbol Device:C
- added C10, C13, C9: 470p, Capacitor_SMD:C_0805_2012Metric, symbol Device:C_US
- added C2: 100nF, Capacitor_SMD:C_0805_2012Metric, symbol Device:C
- added J2: Screw_Terminal_01x02, TerminalBlock_Phoenix:TerminalBlock_Phoenix_MKDS-3-2-5.08_1x02_P5.08mm_Horizontal, symbol Connector:Screw_Terminal_01x02
- added Q7: IXTX110N20L2, Package_TO_SOT_THT:TO-247-3_Vertical, symbol Transistor_FET:Q_NMOS_GDS
- added R10, R15, R16, R21, R3, R4, R9: 100k, Resistor_SMD:R_0805_2012Metric, symbol Device:R
- added R13: 100, Resistor_SMD:R_0805_2012Metric, symbol Device:R_US
- added R19, R23: 0.05, Resistor_SMD:R_2512_6332Metric, symbol Device:R_US
- added U1: R-78HE5.0-0.3, footprints:SIP900W75P254L1200H1300Q3, symbol R-78HE5.0-0.3:R-78HE5.0-0.3
- C11: value 1u -> 470p
- C7: value 470p -> 1uF
- C8: renamed from C9; value 1u -> 1uF
- J1: footprint TerminalBlock_Phoenix:TerminalBlock_Phoenix_MKDS-1,5-2_1x02_P5.00mm_Horizontal -> TerminalBlock_Phoenix:TerminalBlock_Phoenix_MKDS-3-2-5.08_1x02_P5.08mm_Horizontal
- R17: value 1 -> 100; footprint Resistor_SMD:R_2512_6332Metric -> Resistor_SMD:R_0805_2012Metric
- R2, R6: value 100 -> 0.05; footprint Resistor_SMD:R_0805_2012Metric -> Resistor_SMD:R_2512_6332Metric
- R22: value 1k -> 100k; footprint (none) -> Resistor_SMD:R_0805_2012Metric
- R7: value 0.05 -> 100; footprint Resistor_SMD:R_2512_6332Metric -> Resistor_SMD:R_0805_2012Metric
- renumbered C10 to C12, C12 to C14, Q7 to Q6, R13 to R14, R15 to R18, R14 to R20, R16 to R24
Connections:
- net SCK_L is gone; now on an unnamed net: R22.2
- net 5V_LOAD: now also C2.1, C3.1, C4.1, U1.3 (+VOUT); no longer R22.1
- net GND: now also C7.1, IC1.11 (V-), IC2.11 (V-), J1.1 (Pin_1), R2.2, R22.1, R6.2, C1.2, C2.2, C3.2, C4.2, J2.1 (Pin_1), R10.2, R15.2, R16.2, R19.2, R21.1, R23.2, R3.1, R4.1, R9.2, U1.2 (GND); no longer C11.2, J1.2 (Pin_2), R7.2
- net at IC1.1 (OUT_A): now also R11.1, C9.2; no longer R2.1
- net at C6.2, R8.1: now also IC2.7 (OUTB); no longer IC1.14 (OUT_D)
- net at Q1.3 (S), R1.1: now also C5.1, IC1.6 (-INB); no longer IC1.2 (-IN_A)
- net at Q2.3 (S): now also C6.1, IC2.6 (-INB), R2.1; no longer IC1.6 (-INB)
- net at IC1.7 (OUTB): now also C5.2, R7.1
- net at Q3.3 (S), R5.1: now also IC1.2 (-IN_A), C9.1; no longer C5.1, IC1.9 (-INC)
- net at R17.2: now also Q7.1 (G), R21.2; no longer J1.1 (Pin_1)
- net at IC2.2 (-IN_A): now also Q4.3 (S), R6.1, C10.1
- net at R8.2: now also Q2.1 (G), R4.2; no longer Q4.1 (G)
- net at Q3.1 (G): now also R11.2, R9.1; no longer R6.2
- net at R12.2: now also Q4.1 (G), R10.1
- net at IC2.1 (OUT_A), R12.1: now also C10.2
- net at Q6.1 (G), R14.2: now also R16.1
- net at Q5.1 (G): now also R13.2, R15.1; no longer R11.2
- net at Q1.1 (G): now also R7.2, R3.2; no longer R2.2
- net +12V renamed 12V
- net 12V: now also C7.2, C1.1, J2.2 (Pin_2), U1.1 (+VIN)
- removed net -12V: C11.1, IC1.11 (V-), IC2.11 (V-)
- net Vref renamed VREF
- net Vturb renamed VTURB
- net VTURB: now also J1.2 (Pin_2), Q7.2 (D); no longer R17.1
- new net: C13.1, IC1.9 (-INC), Q7.3 (S), R23.1
- new net: C11.2, IC1.14 (OUT_D), R13.1
- new net: C11.1, IC1.13 (-IN_D), Q5.3 (S), R19.1
- new net: C13.2, IC1.8 (OUTC), R17.1
- no-connect marks 7 -> 0
Other:
- added sheet DAC (dac.kicad_sch)
- note removed: "VREF_DAC needs to be divide by 8. 2.048V full scale becomes 0.256V -> (6.98k/1k divider)"
