File: HSWET_PCB.kicad_pcb (KiCad board)
At the start: 2 copper layers, 36 parts, among them J1 TURBINE_IN, J10 arduino enc, J11 turbine pwr, J12 LOAD_OUT, J2 emergency stop, J4 turbine bus, J5 5v, J7 4.5v, J8 GND, J9 arduino lin act, U1 INA238, U2 LTC3525ESC6-5-TRMPBF, U3 YAAJ_DCDC_StepDown_LM2596, U4 LTC3525ESC6-5-TRMPBF

Commit message: part choices, footprints, 3d models, and fixing issues in schematic
Parts:
- removed J10: arduino enc, Connector_PinHeader_1.00mm:PinHeader_1x01_P1.00mm_Vertical
- removed J11: turbine pwr, Connector_PinHeader_1.00mm:PinHeader_1x01_P1.00mm_Vertical
- removed J12: LOAD_OUT, Connector_AMASS:AMASS_XT30PW-M_1x02_P2.50mm_Horizontal
- removed J7: 4.5v, Connector_PinHeader_1.00mm:PinHeader_1x01_P1.00mm_Vertical
- removed J8: GND, Connector_PinHeader_1.00mm:PinHeader_1x01_P1.00mm_Vertical
- removed J9: arduino lin act, Connector_PinHeader_1.00mm:PinHeader_1x01_P1.00mm_Vertical
- removed L2: SRN3015-100M, footprints:SRN3015
- added A1: Arduino_Nano_Every, Module:Arduino_Nano, F.Cu at (120.6, 110.0)
- added C10: 0.22F, Capacitor_SMD:C_0603_1608Metric, F.Cu at (114.5, 142.1)
- added C11: 0.22F, Capacitor_SMD:C_0603_1608Metric, F.Cu at (114.5, 144.6)
- added C12: 10uF, Capacitor_SMD:C_0603_1608Metric, F.Cu at (114.5, 147.1)
- added C13: C, Capacitor_SMD:C_0603_1608Metric, F.Cu at (114.5, 149.6)
- added D4: D_Schottky, footprints:DIOM5436X330N, F.Cu at (138.7, 138.6)
- added D5: BAT54C, Package_TO_SOT_SMD:SOT-23, F.Cu at (137.1, 143.5)
- added F1: MF-MSMF050-2, footprints:FUSM4632X85, F.Cu at (168.4, 123.8)
- added H1: MountingHole_Pad, MountingHole:MountingHole_2.5mm_Pad, F.Cu at (135.1, 89.8)
- added H2: MountingHole_Pad, MountingHole:MountingHole_2.5mm_Pad, F.Cu at (135.1, 96.4)
- added H3: MountingHole_Pad, MountingHole:MountingHole_2.5mm_Pad, F.Cu at (135.1, 102.9)
- added H4: MountingHole_Pad, MountingHole:MountingHole_2.5mm_Pad, F.Cu at (135.1, 109.5)
- added J3: LOAD_OUT, Connector_AMASS:AMASS_XT30PW-M_1x02_P2.50mm_Horizontal, F.Cu at (67.7, 72.5)
- added J6: emergency stop, Connector_JST:JST_EH_B2B-EH-A_1x02_P2.50mm_Vertical, F.Cu at (75.0, 78.0)
- added JP1: Jumper_2_Bridged, Connector_PinHeader_2.54mm:PinHeader_1x02_P2.54mm_Vertical, F.Cu at (134.1, 127.6)
- added PS1: TSR1-4850WI, footprints:CONV_TSR1-4850WI, F.Cu at (91.0, 96.0)
- added Q1: 2N7002, Package_TO_SOT_SMD:SOT-23, F.Cu at (123.0, 143.6)
- added R1: 150k, Resistor_SMD:R_0603_1608Metric, F.Cu at (74.0, 90.0)
- added R14: 309k, Resistor_SMD:R_0603_1608Metric, F.Cu at (118.5, 137.1)
- added R15: 100k, Resistor_SMD:R_0603_1608Metric, F.Cu at (118.5, 139.6)
- added R16: 10k, Resistor_SMD:R_0603_1608Metric, F.Cu at (118.5, 142.1)
- added R17: 787K, Resistor_SMD:R_0603_1608Metric, F.Cu at (118.5, 144.6)
- added R18: 100k, Resistor_SMD:R_0603_1608Metric, F.Cu at (118.5, 147.1)
- added R19: R, Resistor_SMD:R_0603_1608Metric, F.Cu at (132.6, 137.1)
- added R2: 10k, Resistor_SMD:R_0603_1608Metric, F.Cu at (74.0, 87.0)
- added R20: R, Resistor_SMD:R_0603_1608Metric, F.Cu at (132.6, 139.6)
- added R21: 100k, Resistor_SMD:R_0603_1608Metric, F.Cu at (132.6, 142.1)
- added R22: 3.01 M, Resistor_SMD:R_0603_1608Metric, F.Cu at (132.6, 144.6)
- added R23: 100k, Resistor_SMD:R_0603_1608Metric, F.Cu at (132.6, 147.1)
- added R3: 10k, Resistor_SMD:R_0603_1608Metric, F.Cu at (133.8, 124.0)
- added R4: 10k, Resistor_SMD:R_0603_1608Metric, F.Cu at (137.8, 114.0)
- added R7: 330, Resistor_SMD:R_0603_1608Metric, F.Cu at (137.8, 121.5)
- added R8: 330, Resistor_SMD:R_0603_1608Metric, F.Cu at (137.8, 124.0)
- added SW1: SW_DPDT_x2, footprints:1101A2CQEA, F.Cu at (75.3, 65.0)
- added TP1: TestPoint, TestPoint:TestPoint_Pad_1.0x1.0mm, F.Cu at (139.9, 100.3)
- added TP2: TestPoint, TestPoint:TestPoint_Pad_1.0x1.0mm, F.Cu at (139.9, 103.3)
- added TP3: TestPoint, TestPoint:TestPoint_Pad_1.0x1.0mm, F.Cu at (139.9, 106.4)
- added TP4: TestPoint, TestPoint:TestPoint_Pad_1.0x1.0mm, F.Cu at (142.9, 100.3)
- added TP5: TestPoint, TestPoint:TestPoint_Pad_1.0x1.0mm, F.Cu at (142.9, 103.3)
- added TP6: TestPoint, TestPoint:TestPoint_Pad_1.0x1.0mm, F.Cu at (142.9, 106.4)
- added TP7: TestPoint, TestPoint:TestPoint_Pad_1.0x1.0mm, F.Cu at (146.0, 100.3)
- added TP8: TestPoint, TestPoint:TestPoint_Pad_1.0x1.0mm, F.Cu at (146.0, 103.3)
- added TP9: TestPoint, TestPoint:TestPoint_Pad_1.0x1.0mm, F.Cu at (146.0, 106.4)
- added U5: TLV3012AIDBVR, footprints:SOT95P280X145-6N, F.Cu at (137.8, 148.0)
- C2: value 0.47 -> 100nF; footprint footprints:CAPPRD500W60D1000H3150 -> Capacitor_SMD:C_0603_1608Metric
- C3: value 10u -> 4.7 uF; moved to B.Cu
- C4: value 0.47 -> 4.7uF; footprint footprints:CAPPRD500W60D1000H3150 -> Capacitor_SMD:C_0603_1608Metric; moved to B.Cu
- C5: value 1uF -> 220uF; moved to B.Cu
- C6: value 1uF -> 10uF; moved to B.Cu
- C7: value 0.47F -> 470uF; footprint footprints:CAPPRD500W60D1000H3150 -> Capacitor_SMD:C_0603_1608Metric
- C8: value 0.47F -> 1F; footprint footprints:CAPPRD500W60D1000H3150 -> Capacitor_SMD:C_0603_1608Metric
- C9: value 10u -> 1F
- D1: value STPS120M -> D_TVS; footprint footprints:DIO_STPS1L40M -> Diode_SMD:D_SMB_Handsoldering; moved to B.Cu
- D2: footprint footprints:DIOM4336X265N -> Diode_SMD:D_0201_0603Metric_Pad0.64x0.40mm_HandSolder; moved to B.Cu
- D3: value STPS120M -> D_TVS; footprint footprints:DIO_STPS1L40M -> Diode_SMD:D_0201_0603Metric_Pad0.64x0.40mm_HandSolder
- J1: value TURBINE_IN -> turbine bus; footprint Connector_AMASS:AMASS_XT30PW-M_1x02_P2.50mm_Horizontal -> Connector_PinHeader_2.54mm:PinHeader_1x04_P2.54mm_Vertical
- J2: value emergency stop -> turbine bus; footprint Connector_JST:JST_EH_B2B-EH-A_1x02_P2.50mm_Vertical -> Connector_PinHeader_2.54mm:PinHeader_1x04_P2.54mm_Vertical
- J4: value turbine bus -> TURBINE_IN; footprint Connector_PinHeader_2.54mm:PinHeader_1x04_P2.54mm_Horizontal -> Connector_AMASS:AMASS_XT30PW-M_1x02_P2.50mm_Horizontal
- J5: value 5v -> Screw_Terminal_01x02; footprint Connector_PinHeader_1.00mm:PinHeader_1x01_P1.00mm_Vertical -> footprints:1760510000
- L1: value SRN3015-100M -> 1UH; footprint footprints:SRN3015 -> Inductor_SMD:L_Changjiang_FTC201610D
- R10, R11: value R -> 10k; footprint Resistor_THT:R_Axial_DIN0207_L6.3mm_D2.5mm_P10.16mm_Horizontal -> Resistor_SMD:R_0603_1608Metric
- R12, R9: value 10 -> 10k; footprint Resistor_SMD:R_2512_6332Metric -> Resistor_SMD:R_0603_1608Metric
- R5: value 10k -> 0.01
- R6: value 10k -> 330
- U1: value INA238 -> INA260AIPWR
- U2: value LTC3525ESC6-5-TRMPBF -> R-78HE5.0-0.3; footprint footprints:SC70-SC6_LIT -> footprints:SIP900W75P254L1200H1300Q3
- U3: value YAAJ_DCDC_StepDown_LM2596 -> LTC4425EMSE_TRPBF; footprint footprints:YAAJ_DCDC_StepDown_LM2596 -> footprints:MSOP-12_MSE
- U4: value LTC3525ESC6-5-TRMPBF -> TPS61022RWUR; footprint footprints:SC70-SC6_LIT -> footprints:CONV_TPS61022RWUR
- moved C7 253.5 mm to (165.1, 138.3)
- moved R12 248.9 mm to (165.1, 140.8)
- moved U3 240.9 mm to (123.9, 138.6), turned to 0 degrees
- moved R13 240.6 mm to (165.1, 143.3)
- moved D3 237.5 mm to (166.0, 129.0)
- moved J5 225.5 mm to (162.8, 108.3)
- moved C9 212.8 mm to (114.5, 139.6)
- moved L1 212.0 mm to (126.8, 147.5)
- moved C8 210.2 mm to (114.5, 137.1)
- moved J1 207.5 mm to (140.7, 88.8)
- moved R6 206.2 mm to (137.8, 119.0)
- moved U4 204.9 mm to (123.0, 147.6)
- moved J2 183.6 mm to (145.2, 88.8)
- moved R11 172.2 mm to (80.0, 102.0), turned to -90 degrees
- moved U1 171.1 mm to (78.0, 97.0)
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Connections:
- C1 pad 1: GND -> TURB_DIV
- C1 pad 2: 5V -> GND
- C2 pad 1: Net-(D1-K) -> GND
- C2 pad 2: GND -> 5V
- C3 pad 1: 5V -> VIN
- C4 pad 1: Net-(D1-K) -> VIN
- C5 pad 1: Net-(D1-K) -> 5V_LOGIC
- C6 pad 1: Net-(D3-K) -> 5V_ACT
- C7 pad 1: Net-(D3-K) -> ACT_5V_F
- C8 pad 1: Net-(D3-K) -> VBANK
- C8 pad 2: GND -> VMID
- C9 pad 1: 5V -> VMID
- D1 pad 1: Net-(D1-K) -> VIN
- D1 pad 2: Net-(D1-A) -> GND
- D2 pad 1: VIN -> 5V_ACT
- D2 pad 2: GND -> 5V_LOGIC
- D3 pad 1: Net-(D3-K) -> ACT_5V_F
- D3 pad 2: Net-(D3-A) -> GND
- J1 pad 1: Turbine_PWR -> GND
- J1 pad 2: GND -> ACT_5V_F
- J2 pad 1: Turbine_PWR_Read -> 5V_LOGIC
- J2 pad 2: Turbine_PWR_SAFETY -> Net-(J2-Pin_2)
- J4 pad 2: 6V -> TURB_PWR
- J5 pad 1: 5V -> GND
- L1 pad 1: Net-(D3-K) -> VBANK
- L1 pad 2: Net-(U2-SW) -> Net-(U4-SW)
- R10 pad 1: Turbine_PWR -> 5V
- R10 pad 2: Turbine_PWR_Read -> SDA_INA
- R11 pad 1: Turbine_PWR_Read -> SCL_INA
- R11 pad 2: GND -> 5V
- R12 pad 1: 4.5V_BUCK -> 5V_ACT
- R12 pad 2: Net-(D3-A) -> ACT_SENSE
- R13 pad 1: Net-(U1-ALERT) -> ACT_SENSE
- R13 pad 2: 5V -> GND
- R5 pad 1: 5V -> TURB_PWR
- R5 pad 2: SCL_INA -> TURB_LOAD
- R6 pad 1: SDA_INA -> DAC_SCK
- R6 pad 2: 5V -> Net-(J2-Pin_2)
- R9 pad 1: 4.5V_BUCK -> Net-(U1-ALERT)
- R9 pad 2: Net-(D1-A) -> 5V
- U1 pad 1: Turbine_PWR -> TURB_PWR
- U1 pad 13: (no net) -> unconnected-(U1-NC-Pad13)
- U1 pad 14: Turbine_PWR_Read -> TURB_LOAD
- U1 pad 15: Turbine_PWR_Read -> unconnected-(U1-IN--Pad15)
- U1 pad 16: Turbine_PWR_Read -> unconnected-(U1-IN--Pad16)
- U1 pad 2: Turbine_PWR -> unconnected-(U1-IN+-Pad2)
- U1 pad 3: Turbine_PWR -> unconnected-(U1-IN+-Pad3)
- U2 pad 1: Net-(D3-K) -> VIN
- U2 pad 3: Net-(D3-K) -> 5V_LOGIC
- U3 pad 1: VIN -> VBANK
- U3 pad 2: GND -> VBANK
- U3 pad 3: GND -> Net-(U3-PROG)
- U3 pad 4: 4.5V_BUCK -> 5V_LOGIC
- U4 pad 1: Net-(D1-K) -> GND
- U4 pad 2: GND -> Net-(U4-SW)
- U4 pad 3: Net-(D1-K) -> 5V_LOGIC
- U4 pad 4: 5V -> Net-(U4-FB)
- U4 pad 5: GND -> BOOST_EN
- U4 pad 6: Net-(U4-SW) -> GND
