File: HSWET_PCB.kicad_sch (KiCad schematic)
At the start: 66 parts, among them J1 TURBINE_IN, J12 LOAD_OUT, J2 emergency stop, J3 Barrel_Jack, J4 turbine bus, J5 turbine bus, Q1 2N7002, SW1 SW_DPDT_x2, U1 INA238, U3 R-78HE5.0-0.3, U4 TLV3012AIDBVR, U5 LTC4425EMSE_TRPBF, U6 TPS61022RWUR

Commit message: schematic changes
Parts:
- removed C10, C11: 0.47F, symbol Device:C
- removed C12, C5: 10uF, symbol Device:C
- removed C13: C, symbol Device:C
- removed C2: 4.7 uF, symbol Device:C
- removed C3: 4.7uF, symbol Device:C
- removed C4: 220uF, symbol Device:C
- removed D1, D8: D_TVS, symbol Device:D_TVS
- removed D2: D_Schottky, symbol Device:D_Schottky
- removed D4: BAT54C, Package_TO_SOT_SMD:SOT-23, symbol Diode:BAT54C
- removed J1: TURBINE_IN, Connector_AMASS:AMASS_XT30PW-M_1x02_P2.50mm_Horizontal, symbol Connector_Generic:Conn_01x02
- removed J12: LOAD_OUT, Connector_AMASS:AMASS_XT30PW-M_1x02_P2.50mm_Horizontal, symbol Connector_Generic:Conn_01x02
- removed J2: emergency stop, Connector_JST:JST_EH_B2B-EH-A_1x02_P2.50mm_Vertical, symbol Connector_Generic:Conn_01x02
- removed J3: Barrel_Jack, symbol Connector:Barrel_Jack
- removed L2: 1UH, symbol Device:L
- removed PS1: TSR1-4850WI, TSR1-4850WI:CONV_TSR1-4850WI, symbol TSR1-4850WI:TSR1-4850WI
- removed Q1: 2N7002, Package_TO_SOT_SMD:SOT-23, symbol Transistor_FET:2N7002
- removed R1, R15, R2, R8, R9: R, symbol Device:R
- removed R16, R3, R7: 100k, symbol Device:R
- removed R17: 787K, symbol Device:R
- removed R4: 3.01 M, symbol Device:R
- removed SW1: SW_DPDT_x2, symbol Switch:SW_DPDT_x2
- removed U3: R-78HE5.0-0.3, R-78HE5.0-0.3:SIP900W75P254L1200H1300Q3, symbol R-78HE5.0-0.3:R-78HE5.0-0.3
- removed U4: TLV3012AIDBVR, TLV3012AIDBVR:SOT95P280X145-6N, symbol TLV3012AIDBVR:TLV3012AIDBVR
- removed U5: LTC4425EMSE_TRPBF, LTC4425EMSE_TRPBF:MSOP-12_MSE, symbol LTC4425EMSE_TRPBF:LTC4425EMSE_TRPBF
- removed U6: TPS61022RWUR, TPS61022RWUR:CONV_TPS61022RWUR, symbol TPS61022RWUR:TPS61022RWUR
Other:
- added sheet Charger and boost (charger&boost.kicad_sch)
- added sheet Holdup Control (holdup.kicad_sch)
- added sheet Power Input (powerinput.kicad_sch)
- added sheet Regulators (regulators.kicad_sch)
- note added: "*R_SHUNT value needs to be checked Current + Voltage Sensor IIC addres: 0x40"
- note removed: "*R_SHUNT value needs to be calculated IIC addres: 0x40"
- moved on the sheet: C1, C14, C15, D7, F1, J4, J5, R10, R11, R13, R14, R18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

Commit message: part choices, footprints, 3d models, and fixing issues in schematic
Parts:
- removed C1: 100nF, Capacitor_SMD:C_0603_1608Metric, symbol Device:C
- removed C15: 470uF, symbol Device:C
- removed D7: D_TVS, symbol Device:D_TVS
- removed F1: MF-MSMF050-2, MF-MSMF050-2:FUSM4632X85, symbol MF-MSMF050-2:MF-MSMF050-2
- removed R13, R6: 10k, Resistor_SMD:R_0603_1608Metric, symbol Device:R
- removed R14: 0.01, symbol Device:R
- removed R20, R21: 10k, Resistor_THT:R_Axial_DIN0207_L6.3mm_D2.5mm_P10.16mm_Horizontal, symbol Device:R
- removed U1: INA238, footprints:ina260, symbol INA260AIPWR:INA260AIPWR
- added C2: 100nF, Capacitor_SMD:C_0603_1608Metric, symbol Device:C
- added H1, H2, H3, H4: MountingHole_Pad, MountingHole:MountingHole_2.5mm_Pad, symbol Mechanical:MountingHole_Pad
- added R10, R11, R9: 10k, Resistor_SMD:R_0603_1608Metric, symbol Device:R
- added U1: INA260AIPWR, footprints:ina260, symbol ina260aipwr:INA260AIPWR
- C1: renamed from C14; footprint (none) -> Capacitor_SMD:C_0603_1608Metric
- J1: renamed from J4; footprint Connector_PinHeader_2.54mm:PinHeader_1x04_P2.54mm_Horizontal -> Connector_PinHeader_2.54mm:PinHeader_1x04_P2.54mm_Vertical
- J2: renamed from J5; footprint Connector_PinHeader_2.54mm:PinHeader_1x04_P2.54mm_Horizontal -> Connector_PinHeader_2.54mm:PinHeader_1x04_P2.54mm_Vertical
- JP1: footprint (none) -> Connector_PinHeader_2.54mm:PinHeader_1x02_P2.54mm_Vertical
- R1: renamed from R10; footprint Resistor_THT:R_Axial_DIN0207_L6.3mm_D2.5mm_P10.16mm_Horizontal -> Resistor_SMD:R_0603_1608Metric
- R2: renamed from R11; footprint Resistor_THT:R_Axial_DIN0207_L6.3mm_D2.5mm_P10.16mm_Horizontal -> Resistor_SMD:R_0603_1608Metric
- R3: renamed from R18; footprint Resistor_THT:R_Axial_DIN0207_L6.3mm_D2.5mm_P10.16mm_Horizontal -> Resistor_SMD:R_0603_1608Metric
- R4: renamed from R19; footprint Resistor_THT:R_Axial_DIN0207_L6.3mm_D2.5mm_P10.16mm_Horizontal -> Resistor_SMD:R_0603_1608Metric
- R5: value 10k -> 0.01
- R6: renamed from R27; footprint (none) -> Resistor_SMD:R_0603_1608Metric
- R7: renamed from R28; footprint (none) -> Resistor_SMD:R_0603_1608Metric
- R8: renamed from R29; footprint (none) -> Resistor_SMD:R_0603_1608Metric
- TP1, TP2, TP3, TP4: footprint (none) -> TestPoint:TestPoint_Pad_1.0x1.0mm
- TP5: renamed from TP9; footprint (none) -> TestPoint:TestPoint_Pad_1.0x1.0mm
- TP6: renamed from TP5; footprint (none) -> TestPoint:TestPoint_Pad_1.0x1.0mm
- TP7: renamed from TP6; footprint (none) -> TestPoint:TestPoint_Pad_1.0x1.0mm
- TP8: renamed from TP7; footprint (none) -> TestPoint:TestPoint_Pad_1.0x1.0mm
- TP9: renamed from TP8; footprint (none) -> TestPoint:TestPoint_Pad_1.0x1.0mm
- renumbered A2 to A1
Connections:
- net 5V: now also C2.2, R10.1, R11.2, R9.2, U1.10 (VS); no longer R5.1
- net GND: now also C2.1, H1.1, H2.1, H3.1, H4.1, U1.11 (GND), U1.4 (A1), U1.5 (A0), U1.6 (GND)
- net SCL_INA: now also R11.1, U1.9 (SCL); no longer R5.2
- net SDA_INA: now also R10.2, U1.8 (SDA)
- net TURB_LOAD: now also R5.2, U1.14 (IN-)
- net TURB_PWR: now also R5.1, U1.1 (IN+)
- net Turbine_PWR: now also U1.12 (VBUS)
- new net: R9.1, U1.7 (ALERT)
- no-connect marks 2 -> 20
