File: charger&boost.kicad_sch (KiCad schematic)
At the start: 15 parts, among them Q1 2N7002, U5 LTC4425EMSE_TRPBF, U6 TPS61022RWUR

Commit message: part choices, footprints, 3d models, and fixing issues in schematic
Parts:
- C10: renamed from C16; footprint (none) -> Capacitor_SMD:C_0603_1608Metric
- C11: renamed from C17; footprint (none) -> Capacitor_SMD:C_0603_1608Metric
- C12, C13: footprint (none) -> Capacitor_SMD:C_0603_1608Metric
- C8: renamed from C11; footprint (none) -> Capacitor_SMD:C_0603_1608Metric
- C9: renamed from C10; footprint (none) -> Capacitor_SMD:C_0603_1608Metric
- L1: renamed from L2; footprint (none) -> Inductor_SMD:L_Changjiang_FTC201610D
- R14: renamed from R8; footprint (none) -> Resistor_SMD:R_0603_1608Metric
- R15: renamed from R9; footprint (none) -> Resistor_SMD:R_0603_1608Metric
- R16: renamed from R15; footprint (none) -> Resistor_SMD:R_0603_1608Metric
- R17: footprint (none) -> Resistor_SMD:R_0603_1608Metric
- R18: renamed from R16; footprint (none) -> Resistor_SMD:R_0603_1608Metric
- U3: renamed from U5; footprint LTC4425EMSE_TRPBF:MSOP-12_MSE -> footprints:MSOP-12_MSE
- U4: renamed from U6; footprint TPS61022RWUR:CONV_TPS61022RWUR -> footprints:CONV_TPS61022RWUR
Connections:
- net 5V_LOGIC: no longer C13.1
