File: holdup.kicad_sch (KiCad schematic)
At the start: 8 parts, among them U4 TLV3012AIDBVR

Commit message: part choices, footprints, 3d models, and fixing issues in schematic
Parts:
- D4: renamed from D2; footprint (none) -> footprints:DIOM5436X330N
- R19: renamed from R1; footprint (none) -> Resistor_SMD:R_0603_1608Metric
- R20: renamed from R2; footprint (none) -> Resistor_SMD:R_0603_1608Metric
- R21: renamed from R3; footprint (none) -> Resistor_SMD:R_0603_1608Metric
- R22: renamed from R4; footprint (none) -> Resistor_SMD:R_0603_1608Metric
- R23: renamed from R7; footprint (none) -> Resistor_SMD:R_0603_1608Metric
- U5: renamed from U4; footprint TLV3012AIDBVR:SOT95P280X145-6N -> footprints:SOT95P280X145-6N
- renumbered D4 to D5
