File: powerinput.kicad_sch (KiCad schematic)
At the start: 8 parts, among them J1 TURBINE_IN, J12 LOAD_OUT, J2 emergency stop, J3 Barrel_Jack, SW1 SW_DPDT_x2

Commit message: part choices, footprints, 3d models, and fixing issues in schematic
Parts:
- removed J3: Barrel_Jack, symbol Connector:Barrel_Jack
- added J5: Screw_Terminal_01x02, footprints:1760510000, symbol Connector:Screw_Terminal_01x02
- C3: renamed from C2; footprint (none) -> Capacitor_SMD:C_0603_1608Metric
- C4: renamed from C3; footprint (none) -> Capacitor_SMD:C_0603_1608Metric
- D1: renamed from D8; footprint (none) -> Diode_SMD:D_SMB_Handsoldering
- SW1: footprint (none) -> footprints:1101A2CQEA
- renumbered J12 to J3, J1 to J4, J2 to J6
Connections:
- net 9VIN: now also J5.2 (Pin_2)
- net GND: now also J3.1 (Pin_1), J4.1 (Pin_1), J5.1 (Pin_1); no longer J3.2 (Pin_2), J4.2 (Pin_2)
- net TURB_LOAD: now also J3.2 (Pin_2); no longer J3.1 (Pin_1)
- net TURB_PWR: now also J4.2 (Pin_2); no longer J4.1 (Pin_1)
Other:
- moved on the sheet: J3, J6
