File: regulators.kicad_sch (KiCad schematic)
At the start: 5 parts, among them U3 R-78HE5.0-0.3

Commit message: part choices, footprints, 3d models, and fixing issues in schematic
Parts:
- added C7: 470uF, Capacitor_SMD:C_0603_1608Metric, symbol Device:C
- added D3: D_TVS, Diode_SMD:D_0201_0603Metric_Pad0.64x0.40mm_HandSolder, symbol Device:D_TVS
- added F1: MF-MSMF050-2, footprints:FUSM4632X85, symbol MF-MSMF050-2:MF-MSMF050-2
- added R12, R13: 10k, Resistor_SMD:R_0603_1608Metric, symbol Device:R
- C5: renamed from C4; footprint (none) -> Capacitor_SMD:C_0603_1608Metric
- C6: renamed from C5; footprint (none) -> Capacitor_SMD:C_0603_1608Metric
- D2: renamed from D1; footprint (none) -> Diode_SMD:D_0201_0603Metric_Pad0.64x0.40mm_HandSolder
- PS1: footprint TSR1-4850WI:CONV_TSR1-4850WI -> footprints:CONV_TSR1-4850WI
- U2: renamed from U3; footprint R-78HE5.0-0.3:SIP900W75P254L1200H1300Q3 -> footprints:SIP900W75P254L1200H1300Q3
Connections:
- net 5V_ACT: now also F1.1, R12.1
- net GND: now also C7.2, D3.2 (A2), R13.2
- new net ACT_5V_F: C7.1, D3.1 (A1), F1.2
- new net ACT_SENSE: R12.2, R13.1
