File: varload_fix/varload_v1/varload_v1.kicad_sch (KiCad schematic)
At the start: 51 parts, among them IC1 OPA4197ID, IC2 OPA4197ID, J1 Screw_Terminal_01x02, J2 Screw_Terminal_01x02, Q1 IXTX110N20L2, Q2 IXTX110N20L2, Q3 IXTX110N20L2, Q4 IXTX110N20L2, Q5 IXTX110N20L2, Q6 IXTX110N20L2, Q7 IXTX110N20L2, Q8 IXTX110N20L2, U1 R-78HE5.0-0.3

Commit message: layout
Parts:
- added H1, H2, H3, H4: MountingHole_Pad, MountingHole:MountingHole_3.2mm_M3_Pad, symbol Mechanical:MountingHole_Pad
Connections:
- net GND: now also H1.1, H2.1, H3.1, H4.1
